File: transceiver/hardware/_autosave-transceiver.kicad_pcb (KiCad board)
At the start: 4 copper layers, 40 x 40 mm, 54 parts, among them J2 Conn_Coaxial, J3 Conn_01x04, J4 Conn_01x02, J5 Conn_Coaxial, U2 LR2021, U3 STM32G030K8Tx, U4 MAX-M10S, Y1 32.768KHz, Y3 32MHz 10pF

Commit message: finished transceiver pcb
Routing:
- net GND: vias 362 -> 376
Changed lines of the file:
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@@
+	)
+	(via
+		(at 142.2 102.9)
+		(size 0.6)
+		(drill 0.3)
+		(layers "F.Cu" "B.Cu")
+		(free yes)
+		(net "GND")
 	)
 	(via
@@
 	)
 	(via
+		(at 148.7 96.7)
+		(size 0.6)
+		(drill 0.3)
+		(layers "F.Cu" "B.Cu")
+		(free yes)
+		(net "GND")
+	)
+	(via
 		(at 135.3 123.3)
 		(size 0.6)
@@
 	)
 	(via
+		(at 148.7 99.2)
+		(size 0.6)
+		(drill 0.3)
+		(layers "F.Cu" "B.Cu")
+		(free yes)
+		(net "GND")
+	)
+	(via
 		(at 123.7 128)
 		(size 0.6)
@@
 	)
 	(via
+		(at 149.2 101.3)
+		(size 0.6)
+		(drill 0.3)
+		(layers "F.Cu" "B.Cu")
+		(free yes)
+		(net "GND")
+	)
+	(via
 		(at 131 101)
 		(size 0.6)
@@
 	)
 	(via
+		(at 150.1 100.6)
+		(size 0.6)
+		(drill 0.3)
+		(layers "F.Cu" "B.Cu")
+		(free yes)
+		(net "GND")
+	)
+	(via
 		(at 139.9 113.9)
 		(size 0.6)
@@
 	)
 	(via
+		(at 134 102.9)
+		(size 0.6)
+		(drill 0.3)
+		(layers "F.Cu" "B.Cu")
+		(free yes)
+		(net "GND")
+	)
+	(via
 		(at 150.4 116.2)
 		(size 0.6)
@@
 	)
 	(via
+		(at 148.7 92.9)
+		(size 0.6)
+		(drill 0.3)
+		(layers "F.Cu" "B.Cu")
+		(free yes)
+		(net "GND")
+	)
+	(via
 		(at 123.4 116.7)
 		(size 0.6)
@@
 	)
 	(via
+		(at 139.044527 103.016697)
+		(size 0.6)
+		(drill 0.3)
+		(layers "F.Cu" "B.Cu")
+		(free yes)
+		(net "GND")
+	)
+	(via
 		(at 146.6 121.1)
 		(size 0.6)
@@
 	)
 	(via
+		(at 151.5 101.4)
+		(size 0.6)
+		(drill 0.3)
+		(layers "F.Cu" "B.Cu")
+		(free yes)
+		(net "GND")
+	)
+	(via
 		(at 133.3 98.8)
 		(size 0.6)
@@
 	)
 	(via
+		(at 140.8 102.9)
+		(size 0.6)
+		(drill 0.3)
+		(layers "F.Cu" "B.Cu")
+		(free yes)
+		(net "GND")
+	)
+	(via
 		(at 140.1 115.1)
 		(size 0.6)
@@
 	)
 	(via
+		(at 137.5 102.9)
+		(size 0.6)
+		(drill 0.3)
+		(layers "F.Cu" "B.Cu")
+		(free yes)
+		(net "GND")
+	)
+	(via
 		(at 143.2 91)
 		(size 0.6)
@@
 	)
 	(via
+		(at 148 101.9)
+		(size 0.6)
+		(drill 0.3)
+		(layers "F.Cu" "B.Cu")
+		(free yes)
+		(net "GND")
+	)
+	(via
 		(at 154 91)
 		(size 0.6)
@@
 	)
 	(via
+		(at 132.2 102.8)
+		(size 0.6)
+		(drill 0.3)
+		(layers "F.Cu" "B.Cu")
+		(free yes)
+		(net "GND")
+	)
+	(via
 		(at 125.8 123.3)
 		(size 0.6)
@@
 		(size 0.6)
 		(drill 0.3)
+		(layers "F.Cu" "B.Cu")
+		(free yes)
+		(net "GND")
+	)
+	(via
+		(at 135.8 103)
+		(size 0.6)
+		(drill 0.3)

Commit message: fixed via issues
Routing:
- net GND: vias 376 -> 370
Changed lines of the file:
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@@
-	)
-	(via
-		(at 142.2 102.9)
-		(size 0.6)
-		(drill 0.3)
-		(layers "F.Cu" "B.Cu")
-		(free yes)
-		(net "GND")
 	)
 	(via
@@
 	)
 	(via
-		(at 148.7 96.7)
+		(at 148.6 96.9)
 		(size 0.6)
 		(drill 0.3)
@@
 	)
 	(via
-		(at 134 102.9)
-		(size 0.6)
-		(drill 0.3)
-		(layers "F.Cu" "B.Cu")
-		(free yes)
-		(net "GND")
-	)
-	(via
 		(at 150.4 116.2)
 		(size 0.6)
@@
 	)
 	(via
-		(at 139.044527 103.016697)
-		(size 0.6)
-		(drill 0.3)
-		(layers "F.Cu" "B.Cu")
-		(free yes)
-		(net "GND")
-	)
-	(via
 		(at 146.6 121.1)
 		(size 0.6)
@@
 	)
 	(via
-		(at 140.8 102.9)
-		(size 0.6)
-		(drill 0.3)
-		(layers "F.Cu" "B.Cu")
-		(free yes)
-		(net "GND")
-	)
-	(via
 		(at 140.1 115.1)
 		(size 0.6)
@@
 	)
 	(via
-		(at 137.5 102.9)
-		(size 0.6)
-		(drill 0.3)
-		(layers "F.Cu" "B.Cu")
-		(free yes)
-		(net "GND")
-	)
-	(via
 		(at 143.2 91)
 		(size 0.6)
@@
 	)
 	(via
+		(at 120.3 110)
+		(size 0.6)
+		(drill 0.3)
+		(layers "F.Cu" "B.Cu")
+		(net "GND")
+	)
+	(via
 		(at 128.2 92.6)
 		(size 0.6)
@@
 	)
 	(via
-		(at 132.2 102.8)
-		(size 0.6)
-		(drill 0.3)
-		(layers "F.Cu" "B.Cu")
-		(free yes)
-		(net "GND")
-	)
-	(via
 		(at 125.8 123.3)
 		(size 0.6)
@@
 		(size 0.6)
 		(drill 0.3)
-		(layers "F.Cu" "B.Cu")
-		(free yes)
-		(net "GND")
-	)
-	(via
-		(at 135.8 103)
-		(size 0.6)
-		(drill 0.3)
