File: flight-controller/hardware/flight-controller.kicad_sch (KiCad schematic)
At the start: 0 parts

Commit message: testing pcb pannels
Parts:
- added BOOT1, RESET1: SW_Push, Button_Switch_SMD:SW_Push_SPST_NO_Alps_SKRK, symbol Switch:SW_Push
- added C1: 1uF, Capacitor_SMD:C_0603_1608Metric, symbol Device:C
- added C10, C13: 15pF, Capacitor_SMD:C_0402_1005Metric, symbol Device:C
- added C11, C12, C18, C20, C24, C25, C27, C29, C4, C6, C7, C8: 100nF, Capacitor_SMD:C_0402_1005Metric, symbol Device:C
- added C14, C9: 18pF, Capacitor_SMD:C_0402_1005Metric, symbol Device:C
- added C19, C21, C22, C23: 1uF, Capacitor_SMD:C_0402_1005Metric, symbol Device:C
- added C26, C28: 2.2uF, Capacitor_SMD:C_0402_1005Metric, symbol Device:C
- added C30: 4.7uF, Capacitor_SMD:C_0603_1608Metric, symbol Device:C
- added C5: 10uF, Capacitor_SMD:C_0603_1608Metric, symbol Device:C
- added D1, D2: LED, LED_SMD:LED_0603_1608Metric, symbol Device:LED
- added D3: D_Schottky, Diode_SMD:D_SOD-123, symbol Device:D_Schottky
- added J1: USB_C_Receptacle_USB2.0_14P, Connector_USB:USB_C_Receptacle_HRO_TYPE-C-31-M-12, symbol Connector:USB_C_Receptacle_USB2.0_14P
- added J2, J3, J4, J5: Conn_01x04, Connector_PinHeader_2.54mm:PinHeader_1x04_P2.54mm_Vertical, symbol Connector_Generic:Conn_01x04
- added J6: Conn_01x05, Connector_PinSocket_2.54mm:PinSocket_1x05_P2.54mm_Vertical, symbol Connector_Generic:Conn_01x05
- added J7: Conn_01x02, Connector_PinHeader_2.54mm:PinHeader_1x02_P2.54mm_Vertical, symbol Connector_Generic:Conn_01x02
- added J8, J9: Conn_01x01, Connector_Wire:SolderWirePad_1x01_SMD_1.5x3mm, symbol Connector_Generic:Conn_01x01
- added R1, R2: 5.1K, Resistor_SMD:R_0402_1005Metric, symbol Device:R
- added R13, R15: 1K, Resistor_SMD:R_0402_1005Metric, symbol Device:R
- added R3: 10K, Resistor_SMD:R_0402_1005Metric, symbol Device:R
- added U1: STM32H523RCTx, Package_QFP:LQFP-64_10x10mm_P0.5mm, symbol MCU_ST_STM32H5:STM32H523RCTx
- added U2: LSM6DSV, Package_LGA:LGA-14_3x2.5mm_P0.5mm_LayoutBorder3x4y, symbol Sensor_Motion:LSM6DSM
- added U3: MMC5983MA, Package_LGA:LGA-16_3x3mm_P0.5mm, symbol Flight-Controller_Imports:MMC5983MA
- added U4: BMP384, Package_LGA:Rohm_MLGA010V020A_LGA-10_2x2mm_P0.45mm_LayoutBorder2x3y, symbol Flight-Controller_Imports:BMP384
- added U5: MIC5504-3.3YM5, Package_TO_SOT_SMD:SOT-23-5, symbol Regulator_Linear:MIC5504-3.3YM5
- added Y1: 32.768MHz, Crystal:Crystal_SMD_3215-2Pin_3.2x1.5mm, symbol Device:Crystal
- added Y2: 24MHz, Crystal:Crystal_SMD_3225-4Pin_3.2x2.5mm, symbol Device:Crystal_GND24
Connections:
- new net: D2.2 (A), R13.2
- new net: C22.1, D3.1 (K), U5.1 (VIN), U5.3 (EN)
- new net: D3.2 (A), J1.A4 (VBUS), J1.A9 (VBUS), J1.B4 (VBUS), J1.B9 (VBUS)
- new net: C26.1, U1.62 (VCAP)
- new net: C5.1, U3.10 (CAP)
- new net: D1.2 (A), R15.2
- new net: J1.B5 (CC2), R2.2
- new net: J1.A5 (CC1), R1.1
- new net: C28.1, U1.30 (VCAP)
- new net +3.3V: BOOT1.1, C1.1, C12.1, C18.1, C19.1, C20.1, C21.1, C23.1, C24.1, C25.1, C27.1, C29.1, C30.1, C4.1, C6.1, C7.1, C8.1, J2.1 (Pin_1), J3.1 (Pin_1), J4.1 (Pin_1), J5.1 (Pin_1), J8.1 (Pin_1), R15.1, U1.1 (VBAT), U1.13 (VDDA), U1.19 (VDD), U1.32 (VDD), U1.48 (VDD), U1.64 (VDD), U2.1 (SDO/SA0), U2.10 (OCS_Aux), U2.11 (SDO_Aux), U2.12 (CS), U2.2 (SDX), U2.3 (SCX), U2.5 (VDDIO), U2.8 (VDD), U3.13 (VDDIO), U3.2 (VDD), U3.4 (SPI_CS), U4.1 (VDDIO), U4.10 (VDD), U5.5 (VOUT)
- new net BMP_INT: U4.7 (INT)
- new net BOOT: BOOT1.2, R3.1, U1.60 (BOOT0)
- new net CAM_CS: U1.25 (PC5)
- new net CAM_STAT: U1.14 (PA0)
- new net ESC1: J6.1 (Pin_1)
- new net ESC2: J6.2 (Pin_2)
- new net ESC3: J6.3 (Pin_3)
- new net ESC4: J6.4 (Pin_4)
- new net GND: C1.2, C10.2, C11.1, C12.2, C13.2, C14.2, C18.2, C19.2, C20.2, C21.2, C22.2, C23.2, C24.2, C25.2, C26.2, C27.2, C28.2, C29.2, C30.2, C4.2, C5.2, C6.2, C7.2, C8.2, C9.2, D1.1 (K), D2.1 (K), J1.A1 (GND), J1.A12 (GND), J1.B1 (GND), J1.B12 (GND), J1.SH (SHIELD), J2.2 (Pin_2), J3.2 (Pin_2), J4.2 (Pin_2), J5.2 (Pin_2), J6.5 (Pin_5), J9.1 (Pin_1), R1.2, R2.1, R3.2, RESET1.1, U1.12 (VSSA), U1.18 (VSS), U1.31 (VSS), U1.47 (VSS), U1.63 (VSS), U2.6 (GND), U2.7 (GND), U3.11 (GND), U3.9 (GND), U4.3 (VSS), U4.5 (SDO), U4.8 (VSS), U4.9 (VSS), U5.2 (GND), Y2.2, Y2.4
- new net HSE_IN: C9.1, U1.5 (PH0), Y2.1
- new net HSE_OUT: C14.1, U1.6 (PH1), Y2.3
- new net LMS_INT2: U2.9 (INT2)
- new net LR_BUSY: U1.16 (PA2)
- new net LR_CS: U1.17 (PA3)
- new net LR_D10: U1.35 (PB14)
- new net LR_D11: U1.33 (PB12)
- new net LR_D5: U1.26 (PB0)
- new net LR_D6: U1.27 (PB1)
- new net LR_D7: U1.38 (PC7)
- new net LR_D8: U1.37 (PC6)
- new net LR_D9: U1.36 (PB15)
- new net LR_RST: U1.24 (PC4)
- new net LR_STAT: U1.15 (PA1)
- new net LSE_IN: C10.1, U1.3 (PC14), Y1.1
- new net LSE_OUT: C13.1, U1.4 (PC15), Y1.2
- new net LSM_INT1: U2.4 (INT1)
- new net MISO: U1.22 (PA6)
- new net MMC_INT: U3.15 (INT)
- new net MOSI: U1.23 (PA7)
- new net SCK: U1.21 (PA5)
- new net SCL: U1.58 (PB6), U2.13 (SCL)
- new net SCL1: U3.1 (SCL/SPI_SCK), U4.2 (SCK)
- new net SDA: U1.59 (PB7), U2.14 (SDA)
- new net SDA1: U3.16 (SDA/SPI_SDI), U4.4 (SDI)
- new net SD_CLK: U1.53 (PC12)
- new net SD_CMD: U1.28 (PB2)
- new net SD_D0: U1.34 (PB13)
- new net SD_D1: U1.40 (PC9)
- new net SD_D2: U1.51 (PC10)
- new net SD_D3: U1.52 (PC11)
- new net SD_DET: U1.54 (PD2)
- new net STAT_LED: R13.1
- new net STM32_RST: C11.2, RESET1.2, U1.7 (NRST)
- new net SWCLK: J7.1 (Pin_1), U1.49 (PA14(JTCK)
- new net SWDIO: J7.2 (Pin_2), U1.46 (PA13(JTMS)
- new net UART_RX: J2.4 (Pin_4), J3.4 (Pin_4), J4.4 (Pin_4), J5.4 (Pin_4), U1.42 (PA9)
- new net UART_TX: J2.3 (Pin_3), J3.3 (Pin_3), J4.3 (Pin_3), J5.3 (Pin_3), U1.43 (PA10)
- new net USB_+: J1.A6 (D+), J1.B6 (D+), U1.45 (PA12)
- new net USB_-: J1.A7 (D-), J1.B7 (D-), U1.44 (PA11)
- no-connect marks 0 -> 16
Changed lines of the file:
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@@
 	(generator_version "10.0")
 	(paper "A4")
-	(sheet_instances
-		(path "/"
-			(page "1")
-		)
-	)
-	(embedded_fonts no)
-)

Commit message: finished flight controller pcb
Parts:
- added R4, R5: 1.2K, Resistor_SMD:R_0402_1005Metric, symbol Device:R
- J6: footprint Connector_PinSocket_2.54mm:PinSocket_1x05_P2.54mm_Vertical -> (none)
Connections:
- net LR_BUSY is gone; now on net STAT_LED: U1.16 (PA2)
- net LR_CS is gone; now on net BMP_INT: U1.17 (PA3)
- net LR_D6 is gone; now on net LMS_INT2: U1.27 (PB1)
- net SCL1 is gone; now on net SCL: U3.1 (SCL/SPI_SCK), U4.2 (SCK)
- net SDA1 is gone; now on net SDA: U3.16 (SDA/SPI_SDI), U4.4 (SDI)
- net SD_CMD is gone; now on net LSM_INT1: U1.28 (PB2)
- net +3.3V: now also R4.1, R5.1
- net ESC1: now also U1.41 (PA8)
- net ESC2: now also U1.42 (PA9)
- net ESC3: now also U1.56 (PB4(NJTRST))
- net ESC4: now also U1.57 (PB5)
- net MMC_INT: now also U1.43 (PA10)
- net SCL: now also R4.2
- net SDA: now also R5.2
- net CAM_CS: no longer names the net of U1.25 (PC5)
- net CAM_STAT renamed UART_TX4
- net UART_TX4: now also J4.3 (Pin_3)
- net LR_D10 renamed UART_TX1
- net UART_TX1: now also J2.3 (Pin_3)
- net LR_D11 renamed UART_RX5
- net UART_RX5: now also J3.4 (Pin_4)
- net LR_D5: no longer names the net of U1.26 (PB0)
- net LR_D7 renamed UART_RX6
- net UART_RX6: now also J5.4 (Pin_4)
- net LR_D8 renamed UART_TX6
- net UART_TX6: now also J5.3 (Pin_3)
- net LR_D9 renamed UART_RX1
- net UART_RX1: now also J2.4 (Pin_4)
- net LR_RST: no longer names the net of U1.24 (PC4)
- net LR_STAT renamed UART_RX4
- net UART_RX4: now also J4.4 (Pin_4)
- net MISO: no longer names the net of U1.22 (PA6)
- net MOSI: no longer names the net of U1.23 (PA7)
- net SCK: no longer names the net of U1.21 (PA5)
- net SD_CLK: no longer names the net of U1.53 (PC12)
- net SD_D0 renamed UART_TX5
- net UART_TX5: now also J3.3 (Pin_3)
- net SD_D1: no longer names the net of U1.40 (PC9)
- net SD_D2: no longer names the net of U1.51 (PC10)
- net SD_D3: no longer names the net of U1.52 (PC11)
- net SD_DET: no longer names the net of U1.54 (PD2)
- removed net UART_RX: J2.4 (Pin_4), J3.4 (Pin_4), J4.4 (Pin_4), J5.4 (Pin_4), U1.42 (PA9)
- removed net UART_TX: J2.3 (Pin_3), J3.3 (Pin_3), J4.3 (Pin_3), J5.3 (Pin_3), U1.43 (PA10)
- no-connect marks 16 -> 24
Other:
- moved on the sheet: C18, C19, C20, C21, C24, C25, C26, C27, C28, C29, C30, J8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
