File: flight-controller/hardware/flight-controller.kicad_pcb (KiCad board)
At the start: 2 copper layers, 40 x 40 mm, 55 parts, among them J1 USB_C_Receptacle_USB2.0_14P, J2 Conn_01x04, J3 Conn_01x04, J4 Conn_01x04, J5 Conn_01x04, J6 Conn_01x05, J7 Conn_01x02, J8 Conn_01x01, J9 Conn_01x01, U1 STM32H523RCTx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

Commit message: finished flight controller pcb
Parts:
- added R4: 1.2K, Resistor_SMD:R_0402_1005Metric, F.Cu at (148.3, 106.2)
- added R5: 1.2K, Resistor_SMD:R_0402_1005Metric, F.Cu at (148.3, 105.2)
- moved C9 0.91 mm to (159.5, 99.7)
- moved C14 0.45 mm to (156.3, 96.7), turned to 90 degrees
- moved Y2 0.20 mm to (158.6, 97.1)
- moved C20 0.10 mm to (156.0, 100.3)
- moved C21 0.10 mm to (157.0, 100.3)
- turned R2 to 180 degrees
Connections:
- J2 pad 3: /UART_TX -> /UART_TX1
- J2 pad 4: /UART_RX -> /UART_RX1
- J3 pad 3: /UART_TX -> /UART_TX5
- J3 pad 4: /UART_RX -> /UART_RX5
- J4 pad 3: /UART_TX -> /UART_TX4
- J4 pad 4: /UART_RX -> /UART_RX4
- J5 pad 3: /UART_TX -> /UART_TX6
- J5 pad 4: /UART_RX -> /UART_RX6
- U1 pad 14: /CAM_STAT -> /UART_TX4
- U1 pad 15: /LR_STAT -> /UART_RX4
- U1 pad 16: /LR_BUSY -> /STAT_LED
- U1 pad 17: /LR_CS -> /BMP_INT
- U1 pad 21: /SCK -> unconnected-(U1-PA5-Pad21)
- U1 pad 22: /MISO -> unconnected-(U1-PA6-Pad22)
- U1 pad 23: /MOSI -> unconnected-(U1-PA7-Pad23)
- U1 pad 24: /LR_RST -> unconnected-(U1-PC4-Pad24)
- U1 pad 25: /CAM_CS -> unconnected-(U1-PC5-Pad25)
- U1 pad 26: /LR_D5 -> unconnected-(U1-PB0-Pad26)
- U1 pad 27: /LR_D6 -> /LMS_INT2
- U1 pad 28: /SD_CMD -> /LSM_INT1
- U1 pad 33: /LR_D11 -> /UART_RX5
- U1 pad 34: /SD_D0 -> /UART_TX5
- U1 pad 35: /LR_D10 -> /UART_TX1
- U1 pad 36: /LR_D9 -> /UART_RX1
- U1 pad 37: /LR_D8 -> /UART_TX6
- U1 pad 38: /LR_D7 -> /UART_RX6
- U1 pad 40: /SD_D1 -> unconnected-(U1-PC9-Pad40)
- U1 pad 41: unconnected-(U1-PA8-Pad41) -> /ESC1
- U1 pad 42: /UART_RX -> /ESC2
- U1 pad 43: /UART_TX -> /MMC_INT
- U1 pad 51: /SD_D2 -> unconnected-(U1-PC10-Pad51)
- U1 pad 52: /SD_D3 -> unconnected-(U1-PC11-Pad52)
- U1 pad 53: /SD_CLK -> unconnected-(U1-PC12-Pad53)
- U1 pad 54: /SD_DET -> unconnected-(U1-PD2-Pad54)
- U1 pad 56: unconnected-(U1-PB4(NJTRST)-Pad56) -> /ESC3
- U1 pad 57: unconnected-(U1-PB5-Pad57) -> /ESC4
- U3 pad 1: /SCL1 -> /SCL
- U3 pad 16: /SDA1 -> /SDA
- U4 pad 2: /SCL1 -> /SCL
- U4 pad 4: /SDA1 -> /SDA
Routing:
- net +3.3V: track 0.00 -> 54.4 mm, vias 0 -> 22
- net GND: track 0.00 -> 50.7 mm, vias 0 -> 94
- net /SCL: track 0.00 -> 42.9 mm, vias 0 -> 4
- net /SDA: track 0.00 -> 42.4 mm, vias 0 -> 4
- net /STM32_RST: track 0.00 -> 32.4 mm, vias 0 -> 2
- net /ESC1: track 0.00 -> 24.8 mm, vias 0 -> 1
- net /UART_TX1: track 0.00 -> 24.1 mm, vias 0 -> 1
- net /ESC2: track 0.00 -> 24.1 mm, vias 0 -> 1
- net /USB_+: track 0.00 -> 23.4 mm
- net /BOOT: track 0.00 -> 23.3 mm, vias 0 -> 2
- net /USB_-: track 0.00 -> 23.3 mm
- net /UART_RX1: track 0.00 -> 23.2 mm, vias 0 -> 1
- net /ESC3: track 0.00 -> 22.2 mm, vias 0 -> 1
- net /UART_TX6: track 0.00 -> 21.7 mm, vias 0 -> 1
- net /UART_TX5: track 0.00 -> 21.7 mm
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- added copper zone on F.Cu, net +3.3V
- added copper zone on In1.Cu, net +3.3V
- added copper zone on B.Cu, net GND
- added copper zone on F.Cu, net GND
- added copper zone on In2.Cu, net GND
Other:
- copper layers 2 -> 4
- board text added: "3.3v"
- board text added: "GND"
- board text added: "SWCLK"
- board text added: "SWDIO"
